File: PCB/v2-compact/main-board/power_usb.kicad_sch (KiCad schematic)
At the start: 8 parts, among them J20 USB-C, U21 AP7361C-3.3, U22 USBLC6-2SC6

Commit message: Boards: black solder-mask stackup, GND/3V3 plane pours, ESP32-BlackRaven silkscreen art
- Add a 4-layer stackup with BLACK solder mask to both boards (renders/fab in black).
- Pour the inner reference planes: solid GND on the 'GND' layer and +3V3 on the '3V3' layer,
  both boards (~6500mm2 / ~5500mm2 coverage).
- ESP32-BlackRaven branding on the MAIN front: convert the skeletal-raven line-art and the
  bone-font logo to white F.SilkS polygons (scratchpad/img2silk.py, greedy rectangle decomposition
  since bitmap2component is GUI-only) - raven fills the board (~58x81mm, 2419 polys), logo across
  the bottom by the D-pad. New Art_BlackRaven / Art_Logo footprints in SnowOwl.pretty; injected as
  board text (FootprintLoad chokes on the 2419-poly footprint). Removed the old TFT screen label.
- Main-board power reconciliation (schematic): main is now powered from the shield battery over J1;
  J20 USB-C = S3 data/programming only (VBUS_MAIN, not a supply); redundant main LDO U21 removed.

WIP sync note: the schematic main-power change + the datasheet pinout corrections are NOT yet
re-imported to the .kicad_pcb - that's the next batch (re-import removes U21, folds pinout fixes,
re-fills planes). Silkscreen art currently overlaps some pads (buttons/J1/J31) - fab clips silk off
pads, but a clean pass should mask the art away from pads.
Parts:
- removed U21: AP7361C-3.3, Package_TO_SOT_SMD:SOT-23-5, symbol Regulator_Linear:AP7361C-33E
- added R22: 100k, Resistor_SMD:R_0402_1005Metric, symbol Device:R
Connections:
- net +5V: no longer J20.A4 (VBUS), J20.A9 (VBUS), J20.B4 (VBUS), J20.B9 (VBUS), U22.5 (VBUS)
- net GND: now also R22.2
- new net VBUS_MAIN: J20.A4 (VBUS), J20.A9 (VBUS), J20.B4 (VBUS), J20.B9 (VBUS), R22.1, U22.5 (VBUS)
Other:
- note added: "Powered from shield battery via J1 (+5V/+3V3). J20 = S3 USB data/programming only; charge on shield J50."

Commit message: Single USB-C + battery power; J1 vertical on the left edge; U30 model; back-side comments
Power/architecture:
- Remove J50 (the RV1106's own USB-C). The device now has ONE USB-C: the main board's J20.
  J20's VBUS is carried over J1 pin19 (was SPARE) to the shield's BQ25896 charger, so charging +
  the ESP32-S3 data/programming share the single port. Everything runs off the battery.
- Reconcile the nets: J20 VBUS -> VBUS (was VBUS_MAIN), charger VBUS <- J1 pin19, RV1106 keeps its
  microSD (J51) but loses its USB port (reached over UART on J1). Removed orphans R95/R96 (J50 CC
  resistors) and the redundant main LDO U21. Verified: J1 mates 20/20 on both boards, VBUS spans
  J20 -> J1 -> U55, GND healthy (106/37 nodes), no bad net merges.

Placement:
- J1 stack header: was horizontal mid-board, now VERTICAL on the WEST edge at the same spot on both
  boards (they still mate). Nudged the shield's PN532/flash/HTRC (U7/U12/U8) east to clear it, and
  the main's screen east. Status LEDs D10/D11 pulled off the corner mounting holes. 0 real overlaps.

3D + silk:
- U30 (RV1106 Core1106): no KiCad model exists for the Luckfox SoM -> add a sized VRML module
  stand-in (SnowOwl.3dshapes/RV1106_Core1106.wrl; sizes pre-divided by 2.54 for KiCad's inch-unit
  VRML reader). USB-C model: swap the vertical USB4085 for the 16-pin horizontal USB4105 so it
  seats correctly against the horizontal HRO footprint.
- ESP32-BlackRaven art: logo moved to the top by the LEDs, raven dropped down to fill the board.
  Dropped the cluttering TFT label (fab outline kept). Added five back-side silkscreen comments on
  the main board (title/rev, battery, power path, USB-C role, J1 purpose).

Deferred (SWIG pcbnew geometry calls are failing in this environment right now): re-pour the inner
GND/+3V3 planes (inner layers, not visible in renders); apply the datasheet pinout/value fixes to
the power ICs (BQ25896/TPS63020/TPS61230A/MAX17048).
Connections:
- net VBUS_MAIN renamed VBUS
Other:
- note added: "The single USB-C. S3 USB data/programming + charge input: VBUS goes over J1 pin19 to the shield charger. Main runs from the shield battery (+5V/+3V3 via J1)."
- note removed: "Powered from shield battery via J1 (+5V/+3V3). J20 = S3 USB data/programming only; charge on shield J50."
