File: PCB/v2-compact/main-board/stack_header_main.kicad_sch (KiCad schematic)
At the start: 1 part, among them J1 STACK_2x10

Commit message: Single USB-C + battery power; J1 vertical on the left edge; U30 model; back-side comments
Power/architecture:
- Remove J50 (the RV1106's own USB-C). The device now has ONE USB-C: the main board's J20.
  J20's VBUS is carried over J1 pin19 (was SPARE) to the shield's BQ25896 charger, so charging +
  the ESP32-S3 data/programming share the single port. Everything runs off the battery.
- Reconcile the nets: J20 VBUS -> VBUS (was VBUS_MAIN), charger VBUS <- J1 pin19, RV1106 keeps its
  microSD (J51) but loses its USB port (reached over UART on J1). Removed orphans R95/R96 (J50 CC
  resistors) and the redundant main LDO U21. Verified: J1 mates 20/20 on both boards, VBUS spans
  J20 -> J1 -> U55, GND healthy (106/37 nodes), no bad net merges.

Placement:
- J1 stack header: was horizontal mid-board, now VERTICAL on the WEST edge at the same spot on both
  boards (they still mate). Nudged the shield's PN532/flash/HTRC (U7/U12/U8) east to clear it, and
  the main's screen east. Status LEDs D10/D11 pulled off the corner mounting holes. 0 real overlaps.

3D + silk:
- U30 (RV1106 Core1106): no KiCad model exists for the Luckfox SoM -> add a sized VRML module
  stand-in (SnowOwl.3dshapes/RV1106_Core1106.wrl; sizes pre-divided by 2.54 for KiCad's inch-unit
  VRML reader). USB-C model: swap the vertical USB4085 for the 16-pin horizontal USB4105 so it
  seats correctly against the horizontal HRO footprint.
- ESP32-BlackRaven art: logo moved to the top by the LEDs, raven dropped down to fill the board.
  Dropped the cluttering TFT label (fab outline kept). Added five back-side silkscreen comments on
  the main board (title/rev, battery, power path, USB-C role, J1 purpose).

Deferred (SWIG pcbnew geometry calls are failing in this environment right now): re-pour the inner
GND/+3V3 planes (inner layers, not visible in renders); apply the datasheet pinout/value fixes to
the power ICs (BQ25896/TPS63020/TPS61230A/MAX17048).
Connections:
- net SPARE renamed VBUS
Changed lines of the file:
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@@
   (symbol (lib_id "power:+5V") (at 109.22 90.17 0) (unit 1)
     (in_bom yes) (on_board yes) (dnp no)
-    (property "Reference" "#PWR8178292" (at 111.76 87.63 0) (effects (font (size 1.27 1.27)) hide))
+    (property "Reference" "#PWR260FB49" (at 111.76 87.63 0) (effects (font (size 1.27 1.27)) hide))
     (property "Value" "+5V" (at 111.76 92.71 0) (effects (font (size 1.27 1.27))))
     (property "Footprint" "" (at 109.22 90.17 0) (effects (font (size 1.27 1.27)) hide))
     (pin "1")
-    (instances (project "SnowOwl-Main" (path "/a1b2c3d4-0001-4001-8001-000000000015" (reference "#PWR8178292") (unit 1))))
+    (instances (project "SnowOwl-Main" (path "/a1b2c3d4-0001-4001-8001-000000000015" (reference "#PWR260FB49") (unit 1))))
   )
   (wire (pts (xy 127 90.17) (xy 132.08 90.17)) (stroke (width 0) (type default)))
   (symbol (lib_id "power:+3V3") (at 132.08 90.17 0) (unit 1)
     (in_bom yes) (on_board yes) (dnp no)
-    (property "Reference" "#PWR19D2BA2" (at 134.62 87.63 0) (effects (font (size 1.27 1.27)) hide))
+    (property "Reference" "#PWRC9BB6D6" (at 134.62 87.63 0) (effects (font (size 1.27 1.27)) hide))
     (property "Value" "+3V3" (at 134.62 92.71 0) (effects (font (size 1.27 1.27))))
     (property "Footprint" "" (at 132.08 90.17 0) (effects (font (size 1.27 1.27)) hide))
     (pin "1")
-    (instances (project "SnowOwl-Main" (path "/a1b2c3d4-0001-4001-8001-000000000015" (reference "#PWR19D2BA2") (unit 1))))
+    (instances (project "SnowOwl-Main" (path "/a1b2c3d4-0001-4001-8001-000000000015" (reference "#PWRC9BB6D6") (unit 1))))
   )
   (wire (pts (xy 114.3 92.71) (xy 109.22 92.71)) (stroke (width 0) (type default)))
   (symbol (lib_id "power:GND") (at 109.22 92.71 0) (unit 1)
     (in_bom yes) (on_board yes) (dnp no)
-    (property "Reference" "#PWR77F02E6" (at 111.76 90.17 0) (effects (font (size 1.27 1.27)) hide))
+    (property "Reference" "#PWR95549F0" (at 111.76 90.17 0) (effects (font (size 1.27 1.27)) hide))
     (property "Value" "GND" (at 111.76 95.25 0) (effects (font (size 1.27 1.27))))
     (property "Footprint" "" (at 109.22 92.71 0) (effects (font (size 1.27 1.27)) hide))
     (pin "1")
-    (instances (project "SnowOwl-Main" (path "/a1b2c3d4-0001-4001-8001-000000000015" (reference "#PWR77F02E6") (unit 1))))
+    (instances (project "SnowOwl-Main" (path "/a1b2c3d4-0001-4001-8001-000000000015" (reference "#PWR95549F0") (unit 1))))
   )
   (wire (pts (xy 127 92.71) (xy 132.08 92.71)) (stroke (width 0) (type default)))
@@
   (symbol (lib_id "power:GND") (at 132.08 95.25 0) (unit 1)
     (in_bom yes) (on_board yes) (dnp no)
-    (property "Reference" "#PWRFE2D5D8" (at 134.62 92.71 0) (effects (font (size 1.27 1.27)) hide))
+    (property "Reference" "#PWRA397A1F" (at 134.62 92.71 0) (effects (font (size 1.27 1.27)) hide))
     (property "Value" "GND" (at 134.62 97.79 0) (effects (font (size 1.27 1.27))))
     (property "Footprint" "" (at 132.08 95.25 0) (effects (font (size 1.27 1.27)) hide))
     (pin "1")
-    (instances (project "SnowOwl-Main" (path "/a1b2c3d4-0001-4001-8001-000000000015" (reference "#PWRFE2D5D8") (unit 1))))
+    (instances (project "SnowOwl-Main" (path "/a1b2c3d4-0001-4001-8001-000000000015" (reference "#PWRA397A1F") (unit 1))))
   )
   (wire (pts (xy 114.3 97.79) (xy 109.22 97.79)) (stroke (width 0) (type default)))
@@
   (symbol (lib_id "power:GND") (at 132.08 100.33 0) (unit 1)
     (in_bom yes) (on_board yes) (dnp no)
-    (property "Reference" "#PWR3D43FF2" (at 134.62 97.79 0) (effects (font (size 1.27 1.27)) hide))
+    (property "Reference" "#PWR6F6881D" (at 134.62 97.79 0) (effects (font (size 1.27 1.27)) hide))
     (property "Value" "GND" (at 134.62 102.87 0) (effects (font (size 1.27 1.27))))
     (property "Footprint" "" (at 132.08 100.33 0) (effects (font (size 1.27 1.27)) hide))
     (pin "1")
-    (instances (project "SnowOwl-Main" (path "/a1b2c3d4-0001-4001-8001-000000000015" (reference "#PWR3D43FF2") (unit 1))))
+    (instances (project "SnowOwl-Main" (path "/a1b2c3d4-0001-4001-8001-000000000015" (reference "#PWR6F6881D") (unit 1))))
   )
   (wire (pts (xy 114.3 102.87) (xy 109.22 102.87)) (stroke (width 0) (type default)))
   (symbol (lib_id "power:GND") (at 109.22 102.87 0) (unit 1)
     (in_bom yes) (on_board yes) (dnp no)
-    (property "Reference" "#PWR14B9532" (at 111.76 100.33 0) (effects (font (size 1.27 1.27)) hide))
+    (property "Reference" "#PWR9A32CE8" (at 111.76 100.33 0) (effects (font (size 1.27 1.27)) hide))
     (property "Value" "GND" (at 111.76 105.41 0) (effects (font (size 1.27 1.27))))
     (property "Footprint" "" (at 109.22 102.87 0) (effects (font (size 1.27 1.27)) hide))
     (pin "1")
-    (instances (project "SnowOwl-Main" (path "/a1b2c3d4-0001-4001-8001-000000000015" (reference "#PWR14B9532") (unit 1))))
+    (instances (project "SnowOwl-Main" (path "/a1b2c3d4-0001-4001-8001-000000000015" (reference "#PWR9A32CE8") (unit 1))))
   )
   (wire (pts (xy 127 102.87) (xy 132.08 102.87)) (stroke (width 0) (type default)))
@@
   (symbol (lib_id "power:GND") (at 109.22 107.95 0) (unit 1)
     (in_bom yes) (on_board yes) (dnp no)
-    (property "Reference" "#PWRB365FB8" (at 111.76 105.41 0) (effects (font (size 1.27 1.27)) hide))
+    (property "Reference" "#PWR91AAE9E" (at 111.76 105.41 0) (effects (font (size 1.27 1.27)) hide))
     (property "Value" "GND" (at 111.76 110.49 0) (effects (font (size 1.27 1.27))))
     (property "Footprint" "" (at 109.22 107.95 0) (effects (font (size 1.27 1.27)) hide))
     (pin "1")
-    (instances (project "SnowOwl-Main" (path "/a1b2c3d4-0001-4001-8001-000000000015" (reference "#PWRB365FB8") (unit 1))))
+    (instances (project "SnowOwl-Main" (path "/a1b2c3d4-0001-4001-8001-000000000015" (reference "#PWR91AAE9E") (unit 1))))
   )
   (wire (pts (xy 127 107.95) (xy 132.08 107.95)) (stroke (width 0) (type default)))
@@
     (effects (font (size 1.27 1.27)) (justify left)))
   (wire (pts (xy 114.3 113.03) (xy 109.22 113.03)) (stroke (width 0) (type default)))
-  (global_label "SPARE" (shape bidirectional) (at 109.22 113.03 180) (fields_autoplaced)
+  (global_label "VBUS" (shape bidirectional) (at 109.22 113.03 180) (fields_autoplaced)
     (effects (font (size 1.27 1.27)) (justify right)))
   (wire (pts (xy 127 113.03) (xy 132.08 113.03)) (stroke (width 0) (type default)))
   (symbol (lib_id "power:GND") (at 132.08 113.03 0) (unit 1)
     (in_bom yes) (on_board yes) (dnp no)
-    (property "Reference" "#PWR6CEEE3B" (at 134.62 110.49 0) (effects (font (size 1.27 1.27)) hide))
+    (property "Reference" "#PWR9501F75" (at 134.62 110.49 0) (effects (font (size 1.27 1.27)) hide))
     (property "Value" "GND" (at 134.62 115.57 0) (effects (font (size 1.27 1.27))))
     (property "Footprint" "" (at 132.08 113.03 0) (effects (font (size 1.27 1.27)) hide))
     (pin "1")
-    (instances (project "SnowOwl-Main" (path "/a1b2c3d4-0001-4001-8001-000000000015" (reference "#PWR6CEEE3B") (unit 1))))
+    (instances (project "SnowOwl-Main" (path "/a1b2c3d4-0001-4001-8001-000000000015" (reference "#PWR9501F75") (unit 1))))
   )
   (sheet_instances (path "/" (page "1")))
