File: PCB/v2-compact/shield/SnowOwl-Shield.kicad_pcb (KiCad board)
At the start: 4 copper layers, 70 x 100 mm, 81 parts, among them J1 STACK_2x10, J40 C5_PROG_UART, J50 USB-C, J51 microSD, J91 iButton, Q1 MMBT3904, U1 nRF24L01+, U11 TSOP38238, U12 W25Q128JVSSIQ, U2 nRF24L01+, U3 nRF24L01+, U30 Core1106_RV1106, U4 CC1101, U40 ESP32-C5-WROOM-1U-N16R4, U41 AP7361C-3.3, U42 MCP23S17, U5 CC1200RHBR, U6 SX1262IMLTRT, U7 PN532, U8 HTRC11001T, U9 NEO-M9N, Y50 27.12MHz, Y60 40MHz, Y61 32MHz, Y90 4MHz

Commit message: PCB: place the battery + charger power parts on the shield (south back)
Import and place the 24 new power components on the shield's south-back, below the RV1106
and beside the J50 USB-C charge port: BQ25896 charger (U55), TPS63020 buck-boost (U58),
TPS61230A boost (U59), MAX17048 gauge (U57), DW01 protection (U56), AP7361C LDO (U41),
three inductors (L55/58/59), the JST battery connector (BT50), and their passives.

Upgraded the placement anchoring to a SAME-SHEET rule (a support part only anchors to a spec
IC on its own schematic sheet) instead of the single-point distance heuristic - this keeps
each part in its floorplan zone and handles the multi-IC power sheet correctly.

Shield re-verified: 0 same-side overlaps, 0 cross-side hole collisions, 0 parts too close to a
mounting hole, all 105 parts placed. The battery/charger is now physically on the board.
Parts:
- added BT50: LiPo_2500mAh, JST_PH_S2B-PH-K_1x02_P2.00mm_Horizontal, B.Cu at (36.0, 115.0)
- added C45: 47nF, C_0402_1005Metric, B.Cu at (47.8, 102.6)
- added C46: 1uF, C_0402_1005Metric, B.Cu at (50.8, 110.7)
- added C47: 22uF, C_0402_1005Metric, B.Cu at (50.4, 112.1)
- added C48: 22uF, C_0402_1005Metric, B.Cu at (62.5, 104.3)
- added C49: 22uF, C_0402_1005Metric, B.Cu at (73.2, 103.5)
- added C65: 10uF, C_0402_1005Metric, B.Cu at (91.4, 117.2)
- added C66: 10uF, C_0402_1005Metric, B.Cu at (91.4, 122.8)
- added C67: 100nF, C_0402_1005Metric, B.Cu at (92.0, 121.2)
- added L55: 1uH, L_1210_3225Metric, B.Cu at (45.0, 114.0)
- added L58: 1.5uH, L_1210_3225Metric, B.Cu at (60.0, 114.0)
- added L59: 2.2uH, L_1210_3225Metric, B.Cu at (73.0, 114.0)
- added R40: 1100, R_0402_1005Metric, B.Cu at (49.7, 104.3)
- added R41: 10k, R_0402_1005Metric, B.Cu at (49.7, 108.8)
- added R42: 10k, R_0402_1005Metric, B.Cu at (49.5, 105.9)
- added R43: 10k, R_0402_1005Metric, B.Cu at (47.8, 110.8)
- added R44: 1M, R_0402_1005Metric, B.Cu at (67.8, 110.6)
- added R45: 900k, R_0402_1005Metric, B.Cu at (75.7, 103.6)
- added R46: 100k, R_0402_1005Metric, B.Cu at (75.5, 110.7)
- added U55: BQ25896, QFN-24-1EP_4x4mm_P0.5mm_EP2.5x2.5mm, B.Cu at (45.0, 107.0)
- added U56: DW01A_FS8205, SOT-23-6, B.Cu at (48.0, 120.0)
- added U57: MAX17048, DFN-8-1EP_2x3mm_P0.5mm_EP0.61x2.2mm, B.Cu at (33.0, 107.0)
- added U58: TPS63020, DFN-10-1EP_3x3mm_P0.5mm_EP1.58x2.35mm, B.Cu at (60.0, 107.0)
- added U59: TPS61230A, DFN-10-1EP_3x3mm_P0.5mm_EP1.58x2.35mm, B.Cu at (73.0, 107.0)
- moved U41 40.0 mm to (88.0, 120.0)
- moved R96 26.4 mm to (55.1, 119.3)
- moved R95 23.7 mm to (60.1, 119.2)
- moved C95 17.9 mm to (53.6, 81.4)
- moved R57 17.1 mm to (32.1, 92.7)
- moved C71 17.0 mm to (76.1, 36.8)
- moved C43 16.9 mm to (43.2, 102.3)
- moved C41 16.2 mm to (40.1, 109.2)
- moved R56 15.8 mm to (39.5, 98.6)
- moved C87 15.5 mm to (68.2, 46.4)
- moved C40 15.4 mm to (40.6, 104.2)
- moved C63 13.3 mm to (57.0, 68.4)
- moved Q1 12.4 mm to (48.8, 96.5)
- moved C44 12.0 mm to (41.2, 111.0)
- moved C42 11.8 mm to (44.0, 110.5)
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Connections:
- C40 pad 1: +5V -> VBUS
- C41 pad 1: C5_VDD -> VSYS
- C42 pad 1: C5_VDD -> VBAT
- C43 pad 1: +5V -> CHG_PMID
- C44 pad 1: +3V3 -> CHG_REGN
- C94 pad 1: RV_5V -> +5V
- C95 pad 1: RV_5V -> +5V
- J50 pad A4: RV_5V -> VBUS
- J50 pad A9: RV_5V -> VBUS
- J50 pad B4: RV_5V -> VBUS
- J50 pad B9: RV_5V -> VBUS
- U30 pad 12: RV_5V -> +5V

Commit message: Boards: black solder-mask stackup, GND/3V3 plane pours, ESP32-BlackRaven silkscreen art
- Add a 4-layer stackup with BLACK solder mask to both boards (renders/fab in black).
- Pour the inner reference planes: solid GND on the 'GND' layer and +3V3 on the '3V3' layer,
  both boards (~6500mm2 / ~5500mm2 coverage).
- ESP32-BlackRaven branding on the MAIN front: convert the skeletal-raven line-art and the
  bone-font logo to white F.SilkS polygons (scratchpad/img2silk.py, greedy rectangle decomposition
  since bitmap2component is GUI-only) - raven fills the board (~58x81mm, 2419 polys), logo across
  the bottom by the D-pad. New Art_BlackRaven / Art_Logo footprints in SnowOwl.pretty; injected as
  board text (FootprintLoad chokes on the 2419-poly footprint). Removed the old TFT screen label.
- Main-board power reconciliation (schematic): main is now powered from the shield battery over J1;
  J20 USB-C = S3 data/programming only (VBUS_MAIN, not a supply); redundant main LDO U21 removed.

WIP sync note: the schematic main-power change + the datasheet pinout corrections are NOT yet
re-imported to the .kicad_pcb - that's the next batch (re-import removes U21, folds pinout fixes,
re-fills planes). Silkscreen art currently overlaps some pads (buttons/J1/J31) - fab clips silk off
pads, but a clean pass should mask the art away from pads.
Routing:
- added copper zone on In2.Cu, net +3V3
- added copper zone on In1.Cu, net GND
Changed lines of the file:
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@@
 	)
 	(setup
+		(stackup
+			(layer "F.SilkS" (type "Top Silk Screen"))
+			(layer "F.Paste" (type "Top Solder Paste"))
+			(layer "F.Mask" (type "Top Solder Mask") (color "Black") (thickness 0.01))
+			(layer "F.Cu" (type "copper") (thickness 0.035))
+			(layer "dielectric 1" (type "core") (thickness 0.48) (material "FR4") (epsilon_r 4.5) (loss_tangent 0.02))
+			(layer "In1.Cu" (type "copper") (thickness 0.035))
+			(layer "dielectric 2" (type "prepreg") (thickness 0.48) (material "FR4") (epsilon_r 4.5) (loss_tangent 0.02))
+			(layer "In2.Cu" (type "copper") (thickness 0.035))
+			(layer "dielectric 3" (type "core") (thickness 0.48) (material "FR4") (epsilon_r 4.5) (loss_tangent 0.02))
+			(layer "B.Cu" (type "copper") (thickness 0.035))
+			(layer "B.Mask" (type "Bottom Solder Mask") (color "Black") (thickness 0.01))
+			(layer "B.Paste" (type "Bottom Solder Paste"))
+			(layer "B.SilkS" (type "Bottom Silk Screen"))
+			(copper_finish "ENIG")
+			(dielectric_constraints no)
+		)
 		(pad_to_mask_clearance 0)
 		(allow_soldermask_bridges_in_footprints no)
@@
 		)
 	)
+	(zone
+		(net "GND")
+		(layer "In1.Cu")
+		(hatch edge 0.5)
+		(connect_pads
+			(clearance 0.25)
+		)
+		(min_thickness 0.2)
+		(fill yes
+			(thermal_gap 0.5)
+			(thermal_bridge_width 0.5)
+			(island_removal_mode 0)
+		)
+		(polygon
+			(pts
+				(xy 30.25 30.25) (xy 99.75 30.25) (xy 99.75 129.75) (xy 30.25 129.75)
+			)
+		)
+	)
+	(zone
+		(net "+3V3")
+		(layer "In2.Cu")
+		(hatch edge 0.5)
+		(connect_pads
+			(clearance 0.25)
+		)
+		(min_thickness 0.2)
+		(fill yes
+			(thermal_gap 0.5)
+			(thermal_bridge_width 0.5)
+			(island_removal_mode 0)
+		)
+		(polygon
+			(pts
+				(xy 30.25 30.25) (xy 99.75 30.25) (xy 99.75 129.75) (xy 30.25 129.75)
+			)
+		)
+	)

Commit message: Single USB-C + battery power; J1 vertical on the left edge; U30 model; back-side comments
Power/architecture:
- Remove J50 (the RV1106's own USB-C). The device now has ONE USB-C: the main board's J20.
  J20's VBUS is carried over J1 pin19 (was SPARE) to the shield's BQ25896 charger, so charging +
  the ESP32-S3 data/programming share the single port. Everything runs off the battery.
- Reconcile the nets: J20 VBUS -> VBUS (was VBUS_MAIN), charger VBUS <- J1 pin19, RV1106 keeps its
  microSD (J51) but loses its USB port (reached over UART on J1). Removed orphans R95/R96 (J50 CC
  resistors) and the redundant main LDO U21. Verified: J1 mates 20/20 on both boards, VBUS spans
  J20 -> J1 -> U55, GND healthy (106/37 nodes), no bad net merges.

Placement:
- J1 stack header: was horizontal mid-board, now VERTICAL on the WEST edge at the same spot on both
  boards (they still mate). Nudged the shield's PN532/flash/HTRC (U7/U12/U8) east to clear it, and
  the main's screen east. Status LEDs D10/D11 pulled off the corner mounting holes. 0 real overlaps.

3D + silk:
- U30 (RV1106 Core1106): no KiCad model exists for the Luckfox SoM -> add a sized VRML module
  stand-in (SnowOwl.3dshapes/RV1106_Core1106.wrl; sizes pre-divided by 2.54 for KiCad's inch-unit
  VRML reader). USB-C model: swap the vertical USB4085 for the 16-pin horizontal USB4105 so it
  seats correctly against the horizontal HRO footprint.
- ESP32-BlackRaven art: logo moved to the top by the LEDs, raven dropped down to fill the board.
  Dropped the cluttering TFT label (fab outline kept). Added five back-side silkscreen comments on
  the main board (title/rev, battery, power path, USB-C role, J1 purpose).

Deferred (SWIG pcbnew geometry calls are failing in this environment right now): re-pour the inner
GND/+3V3 planes (inner layers, not visible in renders); apply the datasheet pinout/value fixes to
the power ICs (BQ25896/TPS63020/TPS61230A/MAX17048).
Parts:
- removed J50: USB-C, USB_C_Receptacle_HRO_TYPE-C-31-M-12
- removed R95, R96: 5k1, R_0402_1005Metric
- moved J1 45.9 mm to (33.0, 65.0), turned to 90 degrees
- moved C61 16.8 mm to (56.8, 65.6)
- moved C60 16.0 mm to (57.1, 49.6)
- moved Y90 13.0 mm to (50.2, 95.4)
- moved C91 12.9 mm to (51.3, 83.2)
- moved C12 12.5 mm to (63.9, 51.2)
- moved C90 11.7 mm to (52.4, 89.5)
- moved R50 10.1 mm to (52.8, 62.3)
- moved R51 9.51 mm to (52.6, 66.0)
- moved C50 9.06 mm to (41.7, 66.5)
- moved C51 9.06 mm to (49.0, 69.9)
- moved C52 9.06 mm to (41.2, 64.6)
- moved C53 9.06 mm to (49.1, 68.2)
- moved C55 9.06 mm to (41.9, 58.5)
- moved C56 9.06 mm to (47.2, 57.3)
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Connections:
- J1 pad 19: SPARE -> VBUS
