File: PCB/s3-cell/S3-Cell-Base.kicad_pcb (KiCad board)
At the start: 4 copper layers, 91 x 36 mm, 32 parts, among them J1 USB-C, J2 BATT, J3 SMA, J4 nanoSIM, J5 SMA_GNSS, J6 DF40C-2x10 (stack), SW1 BOOT, SW2 RST, U1 USBLC6-2SC6, U2 TP4056, U3 AP2112-3.3, U4 ESP32-S3-WROOM-1U, U5 BG95-M3, U6 TXB0104

Commit message: Shield UI: 1.14" colour TFT + 5-button D-pad; relocate a mounting hole
- Swap the 0.96" OLED for a 1.14" ST7789 colour IPS TFT (SPI) - represented
  by its 12-pin 0.5mm FPC connector plus a glass outline; drop the I2C
  pull-ups (no longer needed)
- Add a D-pad next to the screen: up / down / left / right + centre Select
  (B3U-1000P low-profile tacts), matching the reference layout
- Shift the ESP32-C5 module to the east end (antenna still north) to make
  room for the bigger screen and the buttons
- Move the second mounting hole off the packed east end (it landed 1.2 mm
  from the GNSS SMA and over the back-side SIM) to centre-north by the stack
  connector; both boards keep identical, aligned hole positions

Placement verified overlap-free on both sides; holes >=4mm from all pads.
Other:
- outline, holes or cut-outs redrawn
Changed lines of the file:
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@@
 	)
 	(gr_circle
-		(center 186 130.5)
-		(end 187.1 130.5)
+		(center 157 104)
+		(end 158.1 104)
 		(stroke
 			(width 0.12)
